File: internationals/imu/imu.kicad_sch (KiCad schematic)
At the start: 15 parts, among them J1 5V-JST-XH-B2B, J2 5V-JST-XH-B2B, J3 5V-JST-XH-B2B, J4 IMU-JST-XH-B4B, J5 BT-UART-JST-XH-B4B, J6 Top-UART-JST-XH-B2B, J7 Breakout-Header-01x04, J8 Breakout-Header-01x04, J9 Breakout-Header-01x04, T1 TFmini-Plus-JST-GH-01x04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

Commit message: pcbs: imu: feat: add buttons to schematics
Parts:
- removed J9: Breakout-Header-01x04, Connector_PinHeader_2.54mm:PinHeader_1x04_P2.54mm_Vertical, symbol Connector:Conn_01x04_Pin
- added J9: Breakout-Header-01x04, Connector_PinHeader_2.54mm:PinHeader_1x02_P2.54mm_Vertical, symbol Connector:Conn_01x02_Pin
- added SW1, SW2: SW_Push, Button_Switch_THT:SW_PUSH_6mm, symbol Switch:SW_Push
Connections:
- net GND: now also SW1.1, SW2.1
- net at U2.8 (7): now also J9.1 (Pin_1); no longer J8.1 (Pin_1)
- net at U2.7 (6): now also J9.2 (Pin_2); no longer J8.2 (Pin_2)
- net at J8.3 (Pin_3): now also U2.18 (27); no longer U2.4 (3)
- net at J8.4 (Pin_4): now also U2.17 (26); no longer U2.3 (2)
- net at U2.19 (28): now also J8.2 (Pin_2)
- net at U2.20 (29): now also J8.1 (Pin_1)
- new net Button1: SW1.2, U2.3 (2)
- new net Button2: SW2.2, U2.4 (3)

Commit message: pcbs: imu: fix: 2 pin instead of 4 pin JST
Parts:
- J9: value Breakout-Header-01x04 -> Breakout-Header-01x02
Changed lines of the file:
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@@
 			)
 		)
-		(property "Value" "Breakout-Header-01x04"
+		(property "Value" "Breakout-Header-01x02"
 			(at 90.17 40.64 0)
 			(effects
