File: internationals/pcbs/power/power.kicad_sch (KiCad schematic)
At the start: 6 parts, among them J1 XT60E-M, J2 XT60E-M, J3 XT30-F, J4 XT30-F, J5 JST-XH-B4B, J6 JST-XH-S4B

Commit message: pcbs: power: feat: add mounting holes to schematics
Parts:
- added H1, H2, H3, H4: MountingHole-M3, MountingHole:MountingHole_3.2mm_M3_Pad_Via, symbol Mechanical:MountingHole
