File: internationals/pcbs/imu/imu.kicad_pcb (KiCad board)
At the start: 2 copper layers, 0 parts

Commit message: pcbs: imu: feat: add completed pcb
Parts:
- added G***: LOGO, LOGO, F.Cu at (69.8, 59.5)
- added G*** (x2): LOGO, LOGO, B.Cu at (100.0, 88.5)
- added H1: MountingHole-M3, MountingHole:MountingHole_3.2mm_M3_Pad_Via, F.Cu at (55.0, 55.0)
- added H10: MountingHole-M3, MountingHole:MountingHole_3.2mm_M3_Pad_Via, F.Cu at (116.5, 64.0)
- added H11: MountingHole-M3, MountingHole:MountingHole_3.2mm_M3_Pad_Via, F.Cu at (137.2, 64.0)
- added H12: MountingHole-M3, MountingHole:MountingHole_3.2mm_M3_Pad_Via, F.Cu at (110.0, 120.0)
- added H13: MountingHole-M3, MountingHole:MountingHole_3.2mm_M3_Pad_Via, F.Cu at (80.0, 120.0)
- added H14: MountingHole-M3, MountingHole:MountingHole_3.2mm_M3_Pad_Via, F.Cu at (80.0, 80.0)
- added H15: MountingHole-M3, MountingHole:MountingHole_3.2mm_M3_Pad_Via, F.Cu at (120.0, 80.0)
- added H2: MountingHole-M3, MountingHole:MountingHole_3.2mm_M3_Pad_Via, F.Cu at (145.0, 55.0)
- added H3: MountingHole-M3, MountingHole:MountingHole_3.2mm_M3_Pad_Via, F.Cu at (55.0, 145.0)
- added H4: MountingHole-M3, MountingHole:MountingHole_3.2mm_M3_Pad_Via, F.Cu at (145.0, 145.0)
- added H5: MountingHole-M3, MountingHole:MountingHole_3.2mm_M3_Pad_Via, F.Cu at (27.7, 70.8)
- added H6: MountingHole-M3, MountingHole:MountingHole_3.2mm_M3_Pad_Via, F.Cu at (172.3, 70.8)
- added H7: MountingHole-M3, MountingHole:MountingHole_3.2mm_M3_Pad_Via, F.Cu at (100.0, 178.0)
- added H8: MountingHole-M3, MountingHole:MountingHole_3.2mm_M3_Pad_Via, F.Cu at (90.0, 100.0)
- added H9: MountingHole-M3, MountingHole:MountingHole_3.2mm_M3_Pad_Via, F.Cu at (110.0, 100.0)
- added J1: 5V-JST-XH-B2B, Connector_JST:JST_XH_B2B-XH-A_1x02_P2.50mm_Vertical, F.Cu at (56.8, 77.2)
- added J2: 5V-JST-XH-B2B, Connector_JST:JST_XH_B2B-XH-A_1x02_P2.50mm_Vertical, F.Cu at (76.2, 145.5)
- added J3: 5V-JST-XH-B2B, Connector_JST:JST_XH_B2B-XH-A_1x02_P2.50mm_Vertical, F.Cu at (56.8, 68.2)
- added J4: IMU-JST-XH-B4B, Connector_JST:JST_XH_B4B-XH-A_1x04_P2.50mm_Vertical, F.Cu at (130.5, 77.5)
- added J5: BT-UART-JST-XH-B4B, Connector_JST:JST_XH_B4B-XH-A_1x04_P2.50mm_Vertical, F.Cu at (66.0, 77.2)
- added J6: Top-UART-JST-XH-B2B, Connector_JST:JST_XH_B2B-XH-A_1x02_P2.50mm_Vertical, F.Cu at (34.3, 74.8)
- added J7: Breakout-Header-01x04, Connector_PinHeader_2.54mm:PinHeader_1x04_P2.54mm_Vertical, F.Cu at (139.5, 121.6)
- added J8: Breakout-Header-01x04, Connector_PinHeader_2.54mm:PinHeader_1x04_P2.54mm_Vertical, F.Cu at (147.1, 124.2)
- added J9: Breakout-Header-01x02, Connector_PinHeader_2.54mm:PinHeader_1x02_P2.54mm_Vertical, F.Cu at (115.5, 122.2)
- added JP1: SolderJumper_2_Bridged, Jumper:SolderJumper-2_P1.3mm_Bridged_RoundedPad1.0x1.5mm, F.Cu at (151.5, 77.5)
- added JP2: SolderJumper_2_Open, Jumper:SolderJumper-2_P1.3mm_Open_RoundedPad1.0x1.5mm, F.Cu at (147.5, 77.5)
- added JP3: SolderJumper_2_Open, Jumper:SolderJumper-2_P1.3mm_Open_RoundedPad1.0x1.5mm, F.Cu at (143.5, 77.5)
- added R1: R, PCM_Resistor_THT_AKL:R_Axial_DIN0204_L3.6mm_D1.6mm_P5.08mm_Horizontal, F.Cu at (111.0, 113.5)
- added R2: R, PCM_Resistor_THT_AKL:R_Axial_DIN0204_L3.6mm_D1.6mm_P5.08mm_Horizontal, F.Cu at (111.0, 111.0)
- added R3: R, PCM_Resistor_THT_AKL:R_Axial_DIN0204_L3.6mm_D1.6mm_P5.08mm_Horizontal, F.Cu at (133.0, 73.5)
- added R4: R, PCM_Resistor_THT_AKL:R_Axial_DIN0204_L3.6mm_D1.6mm_P5.08mm_Horizontal, F.Cu at (129.8, 73.5)
- added SW1: SW_Push, Button_Switch_THT:SW_PUSH_6mm, F.Cu at (54.5, 135.5)
- added SW2: SW_Push, Button_Switch_THT:SW_PUSH_6mm, F.Cu at (145.5, 129.0)
- added T1: TFmini-Plus-JST-GH-01x04, Connector_JST:JST_GH_BM04B-GHS-TBT_1x04-1MP_P1.25mm_Vertical, F.Cu at (110.0, 81.0)
- added T2: TFmini-Plus-JST-GH-01x04, Connector_JST:JST_GH_BM04B-GHS-TBT_1x04-1MP_P1.25mm_Vertical, F.Cu at (119.0, 110.0)
- added T3: TFmini-Plus-JST-GH-01x04, Connector_JST:JST_GH_BM04B-GHS-TBT_1x04-1MP_P1.25mm_Vertical, F.Cu at (90.0, 119.0)
- added T4: TFmini-Plus-JST-GH-01x04, Connector_JST:JST_GH_BM04B-GHS-TBT_1x04-1MP_P1.25mm_Vertical, F.Cu at (81.0, 90.0)
- added U1: CN3903 3.3V, PorridgePi-Personal:CN3903, F.Cu at (83.9, 143.7)
- added U2: RP2040-Zero, PorridgePi-Personal:RP2040-Zero, F.Cu at (127.0, 131.0)
- added kibuzzard-666B0E6A (x2): G***, kibuzzard-666B0E6A, F.Cu at (100.0, 47.5)
- added kibuzzard-66706AEF: G***, kibuzzard-66706AEF, F.Cu at (69.8, 73.0)
- added kibuzzard-66706B28: G***, kibuzzard-66706B28, F.Cu at (58.0, 73.2)
- added kibuzzard-66706B28: G***, kibuzzard-66706B28, F.Cu at (75.0, 149.2)
- added kibuzzard-66706B28: G***, kibuzzard-66706B28, B.Cu at (58.0, 73.0)
- added kibuzzard-66706B28: G***, kibuzzard-66706B28, B.Cu at (75.2, 148.0)
- added kibuzzard-66706BB5: G***, kibuzzard-66706BB5, F.Cu at (100.0, 127.5)
- added kibuzzard-66706BB5: G***, kibuzzard-66706BB5, F.Cu at (72.5, 100.0)
- added kibuzzard-66706BB5: G***, kibuzzard-66706BB5, F.Cu at (127.5, 100.0)
- added kibuzzard-66706BB5: G***, kibuzzard-66706BB5, F.Cu at (100.0, 72.5)
- added kibuzzard-667070EB: G***, kibuzzard-667070EB, B.Cu at (80.5, 143.8)
- added kibuzzard-667070FD: G***, kibuzzard-667070FD, F.Cu at (80.5, 146.2)
- added kibuzzard-6670711B: G***, kibuzzard-6670711B, F.Cu at (151.5, 80.0)
- added kibuzzard-66707123: G***, kibuzzard-66707123, F.Cu at (147.5, 80.0)
- added kibuzzard-66707133: G***, kibuzzard-66707133, F.Cu at (143.5, 80.0)
- added kibuzzard-66707151: G***, kibuzzard-66707151, F.Cu at (147.2, 74.5)
- added kibuzzard-667071A6: G***, kibuzzard-667071A6, F.Cu at (126.9, 60.0)
- added kibuzzard-6670727C: G***, kibuzzard-6670727C, F.Cu at (134.2, 81.8)
- added kibuzzard-6670732F: G***, kibuzzard-6670732F, F.Cu at (123.5, 70.5)
- added kibuzzard-6670732F: G***, kibuzzard-6670732F, F.Cu at (99.9, 112.2)
- added kibuzzard-6670735F: G***, kibuzzard-6670735F, B.Cu at (69.8, 80.0)
- added kibuzzard-667073A4: G***, kibuzzard-667073A4, B.Cu at (134.2, 80.0)
- added kibuzzard-667073EF: G***, kibuzzard-667073EF, B.Cu at (108.5, 108.8)
- added kibuzzard-667073EF: G***, kibuzzard-667073EF, B.Cu at (131.2, 71.0)
- added kibuzzard-66707423: G***, kibuzzard-66707423, B.Cu at (143.2, 132.5)
- added kibuzzard-66707423: G***, kibuzzard-66707423, B.Cu at (56.5, 132.2)
Routing:
- net +3.3V: track 0.00 -> 167.2 mm, vias 0 -> 3
- net I2C0_SDA: track 0.00 -> 133.1 mm, vias 0 -> 1
- net IMU-TX0-Top-RX: track 0.00 -> 129.7 mm
- net IMU-RX0-Top-TX: track 0.00 -> 128.9 mm
- net I2C0_SCL: track 0.00 -> 128.4 mm, vias 0 -> 1
- net (no net): track 0.00 -> 107.7 mm, vias 0 -> 20
- net IMU-TX1: track 0.00 -> 102.2 mm
- net IMU-RX1: track 0.00 -> 98.0 mm
- net Button1: track 0.00 -> 69.2 mm, vias 0 -> 1
- net GP13: track 0.00 -> 62.1 mm, vias 0 -> 2
- net I2C1_SDA: track 0.00 -> 55.0 mm
- net I2C1_SCL: track 0.00 -> 54.5 mm
- net Button2: track 0.00 -> 39.1 mm
- net +5V: track 0.00 -> 35.4 mm, vias 0 -> 12
- net V_IMU: track 0.00 -> 29.4 mm
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- added copper zone on F.Cu, net +5V
- added copper zone on B.Cu, net GND
Other:
- board outline added: 152.6 x 142 mm
- board text added: "13 12 11 10"
- board text added: "26 27 28 29"
- board text added: "JLCJLCJLCJLC"
- board text added: "SCL"
- board text added: "SDA"
- board text added: "Team Gloves Zhou Yikun & Zachary Ang Club Automatica Singapore 2024"
