File: internationals/pcbs/imu/imu-rounded.kicad_pcb (KiCad board)
At the start: 2 copper layers, 152.6 x 142 mm, 69 parts, among them J1 5V-JST-XH-B2B, J2 5V-JST-XH-B2B, J3 5V-JST-XH-B2B, J4 IMU-JST-XH-B4B, J5 BT-UART-JST-XH-B4B, J6 Top-UART-JST-XH-B2B, J7 Breakout-Header-01x04, J8 Breakout-Header-01x04, J9 Breakout-Header-01x02, SW1 SW_Push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

Commit message: pcbs: imu: feat: add pcb with tracks rounded
Routing:
- net I2C1_SDA: track 55.0 -> 57.9 mm
- net +3.3V: track 167.2 -> 165.5 mm
- net IMU-TX0-Top-RX: track 129.7 -> 128.3 mm
- net IMU-RX0-Top-TX: track 128.9 -> 127.6 mm
- net I2C0_SDA: track 133.1 -> 131.9 mm
- net I2C0_SCL: track 128.4 -> 127.5 mm
- net +5V: track 35.4 -> 34.6 mm
- net Button2: track 39.1 -> 38.3 mm
- net IMU-TX1: track 102.2 -> 101.4 mm
- net I2C1_SCL: track 54.5 -> 53.9 mm
- net IMU-RX1: track 98.0 -> 97.5 mm
- net Net-(J7-Pin_4): track 27.0 -> 26.5 mm
- net Net-(J7-Pin_3): track 21.1 -> 20.6 mm
